Commit message: Implementation of Camera sensor instead of LIDAR

File: diffbot_description/urdf/diffbot.urdf (robot description, URDF)
Before this commit: robot diffbot, 9 links, 8 joints
Links:
- added link camera_link, mass 0.1; collision cylinder length=0.03 radius=0.03; visual mesh filename=package://diffbot_description/meshes/sensors/package://diff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 scale=1 1 1
Joints:
- added joint camera_joint: type fixed, parent base_link, child camera_link, origin xyz=0 0 0.03 rpy=0 0 0, axis 0 1 0

File: diffbot_description/urdf/diffbot.urdf.xacro (robot description, xacro)
@@ -45,9 +45,17 @@
                       base_props="${base_props}" >
   </xacro:motor>
-  <!-- Sensors -->
-  <xacro:laser prefix="rplidar" parent_link="base_link"
+  <!-- Lidar Sensor -->
+  <!-- <xacro:laser prefix="rplidar" parent_link="base_link"
                    sensor_prop="${sensor_prop}"
                    enable_gpu="${sensor_prop['laser']['enable_gpu']}">
-  </xacro:laser>
+  </xacro:laser> -->
+  <!-- Camera Sensor -->
+  <xacro:camera_sensor
+      parent_link="base_link"
+      sensor_prop="${sensor_prop}"
+      visualize="true"
+      mesh="package://${package_name}/meshes/sensors/hokuyo.dae">
+    <origin xyz="0 0 0" rpy="0 0 0" />
+  </xacro:camera_sensor>
   <!-- Gazebo -->
   <xacro:gazebo_ros_control robotNamespace="/diffbot">

Commit message: Duckietown models base

File: diffbot_description/urdf/diffbot.urdf (robot description, URDF)
Before this commit: robot diffbot, 10 links, 9 joints
Links:
- link camera_link: geometry collision cylinder length=0.03 radius=0.03; visual mesh filename=package://diffbot_description/meshes/sensors/hokuyo.dae scale=1 1 1
Joints:
- joint camera_joint: origin xyz=0 0 0.03 rpy=0 0 0 -> xyz=0 0 0 rpy=0 0 0

File: diffbot_description/urdf/diffbot.urdf.xacro (robot description, xacro)
@@ -55,5 +55,5 @@
       sensor_prop="${sensor_prop}"
       visualize="true"
-      mesh="package://${package_name}/meshes/sensors/hokuyo.dae">
+      mesh="hokuyo.dae">
     <origin xyz="0 0 0" rpy="0 0 0" />
   </xacro:camera_sensor>
