Commit message: diffbot scale up

File: diffbot_description/urdf/_diffbot.urdf (robot description, URDF)
Before this commit: robot diffbot, 10 links, 9 joints
Links:
- link base_link: geometry collision box size=0.195 0.08 0.005; visual mesh filename=package://diffbot_description/meshes/diffbot/chassis.stl
- link front_left_wheel: geometry collision cylinder length=0.025 radius=0.0331; visual mesh filename=package://diffbot_description/meshes/diffbot/../components/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
- link front_right_wheel: geometry collision cylinder length=0.025 radius=0.0331; visual mesh filename=package://diffbot_description/meshes/diffbot/../components/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
- link left_motor: geometry collision box size=0.07 0.0225 0.0188; visual mesh filename=package://diffbot_description/meshes/diffbot/motor.stl
- link rear_caster_base_link: geometry collision box size=0.04 0.04 0.04; visual mesh filename=package://diffbot_description/meshes/diffbot/caster_base.stl
- link rear_caster_rotation_link: geometry collision box size=0.04 0.04 0.04; visual mesh filename=package://diffbot_description/meshes/diffbot/caster_wheel_s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
- link rear_caster_wheel_link: geometry collision cylinder length=0.01 radius=0.015; visual mesh filename=package://diffbot_description/meshes/diffbot/caster_wheel.s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
- link right_motor: geometry collision box size=0.07 0.0225 0.0188; visual mesh filename=package://diffbot_description/meshes/diffbot/motor.stl
Joints:
- joint camera_joint: origin xyz=0.4 0.0 0.04 rpy=0 0 0 -> xyz=0 0 0 rpy=0 0 0
- joint front_left_wheel_joint: origin xyz=0.09250000000000001 0.3375 -0.085 rpy=0 0 0 -> xyz=0.018500000000000003 0.0675 -0.017 rpy=0 0 0
- joint front_right_wheel_joint: origin xyz=0.09250000000000001 -0.3375 -0.085 rpy=0 0 0 -> xyz=0.018500000000000003 -0.0675 -0.017 rpy=0 0 0
- joint left_motor_joint: origin xyz=0.007500000000000007 0.18875000000000003 -0.085 rpy=0 -0.0 0 -> xyz=0.0015000000000000013 0.037750000000000006 -0.017 rpy=0 -0.0 0
- joint rear_caster_base_joint: axis (none) -> 0 0 1; origin xyz=-0.38 -0.0 0.0225 rpy=0 0 0 -> xyz=-0.076 -0.0 0.0045 rpy=0 0 0
- joint rear_caster_rotation_joint: parent rear_caster_base_link -> base_link
- joint rear_caster_wheel_joint: origin xyz=-0.08 0.0 -0.2 rpy=0 0 0 -> xyz=-0.016 0 -0.04 rpy=0 0 0
- joint right_motor_joint: origin xyz=0.007500000000000007 -0.18875000000000003 -0.085 rpy=0 3.141592653589793 0 -> xyz=0.0015000000000000013 -0.037750000000000006 -0.017 rpy=0 3.141592653589793 0

File: diffbot_description/urdf/diffbot.urdf.xacro (robot description, xacro)
@@ -3,4 +3,5 @@
   <xacro:property name="package_name" value="diffbot_description"/>
   <xacro:property name="robot_name" value="diffbot"/>
+  <xacro:property name="scale_factor" value="5.0"/>
   <xacro:include filename="$(find ${package_name})/urdf/include/common_macros.urdf.xacro" />
   <xacro:include filename="$(find ${package_name})/urdf/include/diffbot_caster_macro.urdf.xacro" />
@@ -20,28 +21,34 @@
   <xacro:footprint wheel_props="${front_wheel_props}" />
   <!-- Base link -->
-  <xacro:base base_prop="${base_props}" mesh="${base_props['base']['mesh']}" >
+  <xacro:base base_prop="${base_props}" mesh="${base_props['base']['mesh']}"
+    scale="${scale_factor} ${scale_factor} ${scale_factor}">
     <origin xyz="0 0 0" rpy="0 0 0" />
   </xacro:base>
   <!-- Back Caster Wheel -->
   <xacro:caster_wheel prefix="rear" reflect="-1"
-                      wheel_props="${caster_wheel_props}">
+                      wheel_props="${caster_wheel_props}"
+                      scale="${scale_factor}" >
   </xacro:caster_wheel>
   <!-- Front Wheels -->
   <xacro:wheel prefix="front_right" reflect="-1"
                       wheel_props="${front_wheel_props}"
-                      base_props="${base_props}" >
+                      base_props="${base_props}"
+                      scale="${scale_factor}" >
   </xacro:wheel>
   <xacro:wheel prefix="front_left" reflect="1"
                       wheel_props="${front_wheel_props}"
-                      base_props="${base_props}" >
+                      base_props="${base_props}"
+                      scale="${scale_factor}" >
   </xacro:wheel>
   <!-- Motors -->
   <xacro:motor prefix="right" reflect="-1"
                       motor_props="${motor_props}"
-                      base_props="${base_props}" >
+                      base_props="${base_props}"
+                      scale="${scale_factor}" >
   </xacro:motor>
   <xacro:motor prefix="left" reflect="1"
                       motor_props="${motor_props}"
-                      base_props="${base_props}" >
+                      base_props="${base_props}"
+                      scale="${scale_factor}" >
   </xacro:motor>
   <!-- Lidar Sensor -->

File: diffbot_description/urdf/include/common_macros.urdf.xacro (robot description, xacro)
@@ -16,10 +16,10 @@
 -->
   <xacro:macro name="wheel"
-               params="prefix reflect wheel_props base_props ">
-  <xacro:property name="pos_x_joint"
-     value="${(base_props['base']['x_size']/2) - wheel_props['x_offset']}"/>
-  <xacro:property name="pos_y_joint"
-    value="${(base_props['base']['y_size']/2) + wheel_props['y_offset'] + (wheel_props['length']/2)}"/>
-  <xacro:property name="pos_z_joint" value="${wheel_props['z_offset']}"/>
+               params="prefix reflect wheel_props base_props scale:='1.0'">
+    <xacro:property name="pos_x_joint"
+      value="${float(scale) * ((base_props['base']['x_size']/2) - wheel_props['x_offset'])}"/>
+    <xacro:property name="pos_y_joint"
+      value="${float(scale) *  ((base_props['base']['y_size']/2) + wheel_props['y_offset'] + (wheel_props['length']/2))}"/>
+    <xacro:property name="pos_z_joint" value="${float(scale) * wheel_props['z_offset']}"/>
     <link name="${prefix}_wheel">
     <xacro:if value="${wheel_props['mesh'] != '' }" >
@@ -27,10 +27,10 @@
         <origin xyz="0.0 0 0" rpy="${pi/2} 0 ${pi/2.0*(reflect - 1)}"/>
         <geometry>
-          <xacro:if value="${wheel_props['scale'] == '' }" >
+          <!-- <xacro:if value="${wheel_props['scale'] == '' }" >
             <mesh filename="package://${package_name}/meshes/${robot_name}/${wheel_props['mesh']}" />
           </xacro:if>
-          <xacro:if value="${wheel_props['scale'] != '' }" >
-            <mesh filename="package://${package_name}/meshes/${robot_name}/${wheel_props['mesh']}" scale="${wheel_props['scale']}" />
-          </xacro:if>
+          <xacro:if value="${wheel_props['scale'] != '' }" > -->
+            <mesh filename="package://${package_name}/meshes/${robot_name}/${wheel_props['mesh']}" scale="${scale} ${scale} ${scale}" />
+          <!-- </xacro:if> -->
         </geometry>
         <material name="dark_grey"/>
@@ -41,5 +41,5 @@
         <origin xyz="0.0 0 0" rpy="${pi/2} 0 0"/>
          <geometry>
-         <cylinder radius="${wheel_props['radius']}" length="${wheel_props['length']}"/>
+            <cylinder radius="${float(scale) * wheel_props['radius']}" length="${float(scale) * wheel_props['length']}"/>
         </geometry>
         <material name="red"/>
@@ -49,5 +49,5 @@
         <origin xyz="0 0 0" rpy="${pi/2} 0 0"/>
         <geometry>
-          <cylinder radius="${wheel_props['radius']}" length="${wheel_props['length']}"/>
+          <cylinder radius="${float(scale) * wheel_props['radius']}" length="${float(scale) * wheel_props['length']}"/>
         </geometry>
       </collision>
@@ -91,10 +91,10 @@
 -->
   <xacro:macro name="motor"
-               params="prefix reflect motor_props base_props ">
+               params="prefix reflect motor_props base_props scale:='1.0'">
   <xacro:property name="pos_x_joint"
-     value="${(base_props['base']['x_size']/2) - motor_props['x_offset']}"/>
+     value="${float(scale) * ((base_props['base']['x_size']/2) - motor_props['x_offset'])}"/>
   <xacro:property name="pos_y_joint"
-    value="${(base_props['base']['y_size']/2) + motor_props['y_offset'] + (motor_props['y_size']/2)}"/>
-  <xacro:property name="pos_z_joint" value="${motor_props['z_offset']}"/>
+    value="${float(scale) * ((base_props['base']['y_size']/2) + motor_props['y_offset'] + (motor_props['y_size']/2))}"/>
+  <xacro:property name="pos_z_joint" value="${float(scale) * motor_props['z_offset']}"/>
     <link name="${prefix}_motor">
     <xacro:if value="${motor_props['mesh'] != '' }" >
@@ -102,10 +102,10 @@
         <origin xyz="0.0 0.0 0.0" rpy="0.0 0 ${pi/2.0*(reflect - 1)}"/>
         <geometry>
-          <xacro:if value="${motor_props['scale'] == '' }" >
-            <mesh filename="package://${package_name}/meshes/${robot_name}/${motor_props['mesh']}" />
-          </xacro:if>
+          <!-- <xacro:if value="${motor_props['scale'] == '' }" > -->
+            <mesh filename="package://${package_name}/meshes/${robot_name}/${motor_props['mesh']}" scale="${scale} ${scale} ${scale}" />
+          <!-- </xacro:if>
           <xacro:if value="${motor_props['scale'] != '' }" >
             <mesh filename="package://${package_name}/meshes/${robot_name}/${motor_props['mesh']}" scale="${motor_props['scale']}"/>
-          </xacro:if>
+          </xacro:if> -->
         </geometry>
         <material name="blue"/>
@@ -116,5 +116,5 @@
         <origin xyz="0.0 0 0" rpy="${pi/2} 0 0"/>
          <geometry>
-          <box size="${motor_props['x_size']} ${motor_props['y_size']} ${motor_props['z_size']}"/>
+          <box size="${float(scale) * motor_props['x_size']} ${float(scale) * motor_props['y_size']} ${float(scale) * motor_props['z_size']}"/>
         </geometry>
         <material name="red"/>
@@ -124,5 +124,5 @@
         <origin xyz="0 0 0" rpy="${pi/2} 0 0"/>
         <geometry>
-          <box size="${motor_props['x_size']} ${motor_props['y_size']} ${motor_props['z_size']}"/>
+          <box size="${float(scale) * motor_props['x_size']} ${float(scale) * motor_props['y_size']} ${float(scale) * motor_props['z_size']}"/>
         </geometry>
       </collision>

File: diffbot_description/urdf/include/common_sensors.xacro (robot description, xacro)
@@ -128,4 +128,5 @@
   <joint name="camera_joint" type="fixed">
     <axis xyz="0 1 0" />
+    <origin xyz="${sensor_prop['camera']['dx']} ${sensor_prop['camera']['dy']} ${sensor_prop['camera']['dz']}" rpy="0 0 0"/>
     <xacro:insert_block name="joint_origin" />
     <parent link="${parent_link}"/>

File: diffbot_description/urdf/include/diffbot_caster_macro.urdf.xacro (robot description, xacro)
@@ -1,47 +1,30 @@
 <?xml version="1.0"?>
 <robot xmlns:xacro="http://www.ros.org/wiki/xacro">
-<!-- ===================== Caster xacro =========================================
-  Xacro to create caster links and the respective joints. For more detail information and usage, see:
-    https://github.com/pxalcantara/mobile_robot_description/wiki/Motor-xacro
-  params:
-  - prefix [string]: used to diferentiate the link and joint name;
-  - reflect [1/-1]: value to set the side of the caster;
-  - wheel_props [dictionary]: wheel properties;
-  - base_props [dictionary]: base link properties;
-  - mesh [string]: file name of the wheel mesh;
-    - DEFAULT Value -> Empty string
--->
-<!-- Caster wheel link & joint macro -->
-  <!-- locationprefix locationright wheel_base_dx TODO remove -->
+  <!-- Caster wheel link & joint macro -->
   <xacro:macro name="caster_wheel"
-                params="prefix reflect wheel_props locationright:=${0} scale:=''">
+               params="prefix reflect wheel_props locationright:=${0} scale:='1.0'">
     <!-- caster base (fixed) -->
     <link name="${prefix}_caster_base_link">
-      <xacro:box_inertia  m="${wheel_props['base']['mass']}"
-                          x="${wheel_props['base']['size']['x']}"
-                          y="${wheel_props['base']['size']['y']}"
-                          z="${wheel_props['base']['size']['z']}"
-                          o_xyz="0.0 0.0 ${-wheel_props['base']['size']['z']/2.0}"
-                          o_rpy="0.0 0.0 0.0" />
-      <xacro:if value="${wheel_props['base']['mesh'] != '' }" >
+      <xacro:box_inertia
+        m="${wheel_props['base']['mass']}"
+        x="${wheel_props['base']['size']['x']}"
+        y="${wheel_props['base']['size']['y']}"
+        z="${wheel_props['base']['size']['z']}"
+        o_xyz="0.0 0.0 ${-wheel_props['base']['size']['z']/2.0}"
+        o_rpy="0.0 0.0 0.0" />
+      <xacro:if value="${wheel_props['base']['mesh'] != ''}">
         <visual>
-          <origin xyz="0 0 ${-wheel_props['base']['size']['z']/2.0}" rpy="0 0 0" />
+          <origin xyz="0 0 ${-scale * wheel_props['base']['size']['z']/2.0}" rpy="0 0 0" />
           <geometry>
-            <xacro:if value="${scale != '' }" >
-              <mesh filename="package://${package_name}/meshes/${robot_name}/${wheel_props['base']['mesh']}" scale="${scale}"/>
-            </xacro:if>
-            <xacro:if value="${scale == '' }" >
-              <mesh filename="package://${package_name}/meshes/${robot_name}/${wheel_props['base']['mesh']}" />
-            </xacro:if>
+            <mesh filename="package://${package_name}/meshes/${robot_name}/${wheel_props['base']['mesh']}" scale="${scale} ${scale} ${scale}" />
           </geometry>
-          <!-- xacro:insert_block name="material_silver" / TODO use this block? -->
           <material name="silver"/>
         </visual>
       </xacro:if>
-      <xacro:if value="${wheel_props['base']['mesh'] == '' }" >
+      <xacro:if value="${wheel_props['base']['mesh'] == ''}">
         <visual>
-          <origin xyz="0 0 ${-wheel_props['base']['size']['z']/2.0}" rpy="0 0 0" />
+          <origin xyz="0 0 ${-scale * wheel_props['base']['size']['z']/2.0}" rpy="0 0 0" />
           <geometry>
-            <box size="${wheel_props['base']['size']['x']} ${wheel_props['base']['size']['y']} ${wheel_props['base']['size']['z']}" />
+            <box size="${scale * wheel_props['base']['size']['x']} ${scale * wheel_props['base']['size']['y']} ${scale * wheel_props['base']['size']['z']}" />
           </geometry>
           <material name="red"/>
@@ -49,17 +32,15 @@
       </xacro:if>
       <collision>
-        <origin xyz="0 0 ${-wheel_props['base']['size']['z']/2.0}" rpy="0 0 0" />
+        <origin xyz="0 0 ${-scale * wheel_props['base']['size']['z']/2.0}" rpy="0 0 0" />
         <geometry>
-          <box size="${wheel_props['base']['size']['x']} ${wheel_props['base']['size']['y']} ${wheel_props['base']['size']['z']}" />
+          <box size="${scale * wheel_props['base']['size']['x']} ${scale * wheel_props['base']['size']['y']} ${scale * wheel_props['base']['size']['z']}" />
         </geometry>
       </collision>
     </link>
     <joint name="${prefix}_caster_base_joint" type="fixed">
-      <origin xyz="${wheel_props['base']['dx']} ${-wheel_props['base']['dy'] * locationright} ${wheel_props['base']['dz']}"
+      <origin xyz="${scale * wheel_props['base']['dx']} ${-scale * wheel_props['base']['dy'] * locationright} ${scale * wheel_props['base']['dz']}"
               rpy="0 0 0" />
       <parent link="base_link" />
       <child link="${prefix}_caster_base_link" />
-      <axis xyz="0 0 1" />
-      <dynamics damping="0.01" friction="0.0"/>
     </joint>
     <gazebo reference="${prefix}_caster_base_link">
@@ -68,30 +49,25 @@
     <!-- caster hub -->
     <link name="${prefix}_caster_rotation_link">
-      <xacro:box_inertia  m="${wheel_props['hub']['mass']}"
-                          x="${wheel_props['hub']['size']['x']}"
-                          y="${wheel_props['hub']['size']['y']}"
-                          z="${wheel_props['hub']['size']['z']}"
-                          o_xyz="0.0 0.0 ${-wheel_props['hub']['size']['z']/2.0}"
-                          o_rpy="0.0 0.0 0.0" />
-      <xacro:if value="${wheel_props['hub']['mesh'] != '' }" >
+      <xacro:box_inertia
+        m="${wheel_props['hub']['mass']}"
+        x="${wheel_props['hub']['size']['x']}"
+        y="${wheel_props['hub']['size']['y']}"
+        z="${wheel_props['hub']['size']['z']}"
+        o_xyz="0.0 0.0 ${-wheel_props['hub']['size']['z']/2.0}"
+        o_rpy="0.0 0.0 0.0" />
+      <xacro:if value="${wheel_props['hub']['mesh'] != ''}">
         <visual>
-          <origin xyz="0 0 ${-wheel_props['hub']['size']['z']/2.0}" rpy="0 0 0" />
+          <origin xyz="0 0 ${-scale * wheel_props['hub']['size']['z']/2.0}" rpy="0 0 0" />
           <geometry>
-            <xacro:if value="${scale != '' }" >
-              <mesh filename="package://${package_name}/meshes/${robot_name}/${wheel_props['hub']['mesh']}" scale="${scale}"/>
-            </xacro:if>
-            <xacro:if value="${scale == '' }" >
-              <mesh filename="package://${package_name}/meshes/${robot_name}/${wheel_props['hub']['mesh']}" />
-            </xacro:if>
+            <mesh filename="package://${package_name}/meshes/${robot_name}/${wheel_props['hub']['mesh']}" scale="${scale} ${scale} ${scale}" />
           </geometry>
-          <!-- xacro:insert_block name="material_silver" / TODO use this block? -->
           <material name="silver"/>
         </visual>
       </xacro:if>
-      <xacro:if value="${wheel_props['hub']['mesh'] == '' }" >
+      <xacro:if value="${wheel_props['hub']['mesh'] == ''}">
         <visual>
-          <origin xyz="0 0 ${-wheel_props['hub']['size']['z']/2.0}" rpy="0 0 0" />
+          <origin xyz="0 0 ${-scale * wheel_props['hub']['size']['z']/2.0}" rpy="0 0 0" />
           <geometry>
-            <box size="${wheel_props['hub']['size']['x']} ${wheel_props['hub']['size']['y']} ${wheel_props['hub']['size']['z']}" />
+            <box size="${scale * wheel_props['hub']['size']['x']} ${scale * wheel_props['hub']['size']['y']} ${scale * wheel_props['hub']['size']['z']}" />
           </geometry>
           <material name="red"/>
@@ -99,7 +75,7 @@
       </xacro:if>
       <collision>
-        <origin xyz="0 0 ${-wheel_props['hub']['size']['z']/2.0}" rpy="0 0 0" />
+        <origin xyz="0 0 ${-scale * wheel_props['hub']['size']['z']/2.0}" rpy="0 0 0" />
         <geometry>
-          <box size="${wheel_props['hub']['size']['x']} ${wheel_props['hub']['size']['y']} ${wheel_props['hub']['size']['z']}" />
+          <box size="${scale * wheel_props['hub']['size']['x']} ${scale * wheel_props['hub']['size']['y']} ${scale * wheel_props['hub']['size']['z']}" />
         </geometry>
       </collision>
@@ -108,39 +84,28 @@
       <origin xyz="${wheel_props['hub']['dx']} ${-wheel_props['hub']['dy'] * locationright} ${wheel_props['hub']['dz']}"
               rpy="0 0 0" />
-      <parent link="base_link" />
+      <parent link="${prefix}_caster_base_link" />
       <child link="${prefix}_caster_rotation_link" />
       <axis xyz="0 0 1" />
-      <dynamics damping="0.01" friction="0.0"/>
     </joint>
-    <gazebo reference="${prefix}_caster_rotation_link">
-      <material>Gazebo/Grey</material>
-    </gazebo>
     <!-- caster wheel -->
     <link name="${prefix}_caster_wheel_link">
-      <xacro:cylinder_inertia m="${wheel_props['wheel']['mass']}"
-                              r="${wheel_props['wheel']['radius']}"
-                              l="${wheel_props['wheel']['length']}">
-        <!-- TODO unused block error?: origin xyz="0 0 0" rpy="${pi/2} 0 0" /-->
-      </xacro:cylinder_inertia>
-      <xacro:if value="${wheel_props['wheel']['mesh'] != '' }" >
+      <xacro:cylinder_inertia
+        m="${wheel_props['wheel']['mass']}"
+        r="${wheel_props['wheel']['radius']}"
+        l="${wheel_props['wheel']['length']}" />
+      <xacro:if value="${wheel_props['wheel']['mesh'] != ''}">
         <visual>
           <origin xyz="0 0 0" rpy="0 0 0" />
           <geometry>
-            <xacro:if value="${scale != '' }" >
-              <mesh filename="package://${package_name}/meshes/${robot_name}/${wheel_props['wheel']['mesh']}" scale="${scale}"/>
-            </xacro:if>
-            <xacro:if value="${scale == '' }" >
-              <mesh filename="package://${package_name}/meshes/${robot_name}/${wheel_props['wheel']['mesh']}" />
-            </xacro:if>
+            <mesh filename="package://${package_name}/meshes/${robot_name}/${wheel_props['wheel']['mesh']}" scale="${scale} ${scale} ${scale}" />
           </geometry>
-          <!-- TODO use this?: xacro:insert_block name="material_dark_grey" /-->
           <material name="black"/>
         </visual>
       </xacro:if>
-      <xacro:if value="${wheel_props['wheel']['mesh'] == '' }" >
+      <xacro:if value="${wheel_props['wheel']['mesh'] == ''}">
         <visual>
           <origin xyz="0 0 0" rpy="${pi/2} 0 0" />
           <geometry>
-            <cylinder length="${wheel_props['wheel']['length']}" radius="${wheel_props['wheel']['radius']}" />
+            <cylinder length="${scale * wheel_props['wheel']['length']}" radius="${scale * wheel_props['wheel']['radius']}" />
           </geometry>
           <material name="red"/>
@@ -150,10 +115,10 @@
         <origin xyz="0 0 0" rpy="${pi/2} 0 0" />
         <geometry>
-          <cylinder length="${wheel_props['wheel']['length']}" radius="${wheel_props['wheel']['radius']}" />
+          <cylinder length="${scale * wheel_props['wheel']['length']}" radius="${scale * wheel_props['wheel']['radius']}" />
         </geometry>
       </collision>
     </link>
     <joint name="${prefix}_caster_wheel_joint" type="continuous">
-      <origin xyz="${wheel_props['wheel']['dx']} ${-wheel_props['wheel']['dy'] * locationright} ${wheel_props['wheel']['dz']}"
+      <origin xyz="${scale * wheel_props['wheel']['dx']} ${-scale * wheel_props['wheel']['dy'] * locationright} ${scale * wheel_props['wheel']['dz']}"
               rpy="0 0 0" />
       <parent link="${prefix}_caster_rotation_link" />
@@ -161,7 +126,4 @@
       <axis xyz="0 1 0" />
     </joint>
-    <gazebo reference="${prefix}_caster_wheel_link">
-      <material>Gazebo/DarkGrey</material>
-    </gazebo>
   </xacro:macro>
 </robot>
